File: resources/Eagle Boards/Baja Spring/main_board.brd (EAGLE design)
At the start: 116.8 x 128.7 mm, 12 parts, among them J1 F-1X18-SIP-100-32, J2 F-1X18-SIP-100-32, J3 RJ45, J4 RJ45

Commit message: mhb
Connections:
- new net BUSY: B1.4, J2.7
Routing:
- net BUSY: track 0.00 -> 95.2 mm
Changed lines of the file:
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@@
 <wire x1="98.1456" y1="92.5068" x2="98.287678125" y2="92.608934375" width="0.1524" layer="1"/>
+</signal>
+<signal name="BUSY">
+<contactref element="J2" pad="7"/>
+<contactref element="B1" pad="4"/>
+<wire x1="78.55" y1="99.83" x2="83.06046875" y2="95.31953125" width="0.1524" layer="16"/>
+<wire x1="83.06046875" y1="95.31953125" x2="92.419328125" y2="95.31953125" width="0.1524" layer="16"/>
+<wire x1="92.419328125" y1="95.31953125" x2="94.475415625" y2="93.26344375" width="0.1524" layer="16"/>
+<wire x1="94.475415625" y1="93.26344375" x2="94.475415625" y2="86.22579375" width="0.1524" layer="16"/>
+<wire x1="94.475415625" y1="86.22579375" x2="99.119371875" y2="81.5818375" width="0.1524" layer="16"/>
+<wire x1="99.119371875" y1="81.5818375" x2="99.119371875" y2="76.35400625" width="0.1524" layer="16"/>
+<wire x1="99.119371875" y1="76.35400625" x2="79.42283125" y2="56.657465625" width="0.1524" layer="16"/>
+<wire x1="79.42283125" y1="56.657465625" x2="68.100665625" y2="56.657465625" width="0.1524" layer="16"/>
+<wire x1="68.100665625" y1="56.657465625" x2="63.614796875" y2="52.171596875" width="0.1524" layer="16"/>
+<wire x1="63.614796875" y1="52.171596875" x2="53.048403125" y2="52.171596875" width="0.1524" layer="16"/>
+<wire x1="53.048403125" y1="52.171596875" x2="51.88" y2="53.34" width="0.1524" layer="16"/>
 </signal>
 </signals>
