File: resources/Eagle Boards/Baja Spring/main_board.sch (EAGLE design)
At the start: 12 parts, among them J1 F-1X18-SIP-100-32, J2 F-1X18-SIP-100-32, J3 RJ45, J4 RJ45

Commit message: mhb
Connections:
- new net BUSY: B1.4, J2.7
Changed lines of the file:
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@@
+</segment>
+</net>
+<net name="BUSY" class="0">
+<segment>
+<pinref part="J2" gate="G$1" pin="7"/>
+<wire x1="48.26" y1="144.78" x2="43.18" y2="144.78" width="0.1524" layer="91"/>
+<label x="40.64" y="144.78" size="1.778" layer="95"/>
+</segment>
+<segment>
+<pinref part="B1" gate="G$1" pin="4"/>
+<wire x1="25.4" y1="27.94" x2="22.86" y2="27.94" width="0.1524" layer="91"/>
+<label x="20.32" y="27.94" size="1.778" layer="95"/>
 </segment>
 </net>
